File: hardware/kicad/hridaymitra.kicad_sch (KiCad schematic)
At the start: 59 parts, among them J1 Electrodes: 4 foot plates + 4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, J10 MT3608 module: IN+ IN- OUT+ O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, J11 AD8232 (optional; off for pac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, J2 MAX30102 module (finger), J3 HX711 module: VCC GND DT SCK, J4 HX711 module: E+ E- A- A+, J5 4 load cells as one bridge, J6 PAM8403 module: 5V GND LIN RI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, J8 SIM800L module: VCC GND TXD R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, J9 TP4056 module: B+ B- OUT+ OUT-, SW1 green button, SW2 red button, SW3 SOS button, SW4 power switch, U1 MCP6002, U2 INA126, U3 74HC4053 (body / R5 select), U4 74HC4052 (current pair), U5 74HC4052 (sense pair), U6 ESP32-WROOM-32 (DevKit), U7 3.3 V LDO (on DevKit)

Commit message: Firmware, offline engine on the ESP32, product features, full flow
- ESP32 stool firmware (check-in, Goertzel impedance, PPG, SMS care loop) and
  ESP32-C3 amulet firmware (breathing, sit-ups, activity, falls, SOS over BLE);
  both compile with arduino-cli
- Alert engine ported to C++ (engine_core.h): 100% identical lights to the
  Python engine over 3,231 patient-days (tests/test_engine_parity.py)
- Product layer: doctor's sick-day plan, coaching tips, two users per stool,
  daily self-test, 11:00 reminder, Sunday ASHA summary, seat vibration,
  tablet drawer, village dashboard, OPD report, ABDM/FHIR export
- Engine: "no check-in" day holds the light; cold-start "learning" flag
- Stool bridge + live dashboard, run.py one-command flow, ML comparator
- Report, pitch deck and script generated from live results; evidence and
  decisions docs; schematic, guides, cost and block diagram updated

Co-Authored-By: Claude Opus 5.5 <noreply@anthropic.com>
Parts:
- added D4: 1N4148 flyback, symbol Device:D
- added M1: coin vibration motor (seat), symbol Motor:Motor_DC
- added Q1: 2N2222 (vibration driver), symbol Device:Q_NPN
- added R20: 10k, symbol Device:R
- added R21: 1k, symbol Device:R
- added SW5: tablet-drawer microswitch, symbol Switch:SW_Push
- J11: value AD8232 (optional; off for pacemaker/ICD) -> AD8232 (optional; off for pacemaker/ICD; LO- unused)
Connections:
- net +3V3: now also R20.1
- net +5V: now also D4.1 (K), M1.1 (+)
- net GND: now also Q1.E, SW5.2
- net VIBRA: now reaches U6.31 (IO19)
- net VIBRA: now also R21.1
- net ECG_LON: no longer names the net of J11.5 (Pin_5)
- net ECG_LON: no longer U6.4 (SENSOR_VP)
- new net DRAWER: R20.2, SW5.1, U6.4 (SENSOR_VP)
- new net VIB_B: Q1.B, R21.2
- new net VIB_C: D4.2 (A), M1.2 (-), Q1.C
