File: hardware/kicad/hridaymitra.kicad_sch (KiCad schematic)
At the start: 65 parts, among them J1 Electrodes: 4 foot plates + 4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, J10 MT3608 module: IN+ IN- OUT+ O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, J11 AD8232 (optional; off for pac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, J2 MAX30102 module (finger), J3 HX711 module: VCC GND DT SCK, J4 HX711 module: E+ E- A- A+, J5 4 load cells as one bridge, J6 PAM8403 module: 5V GND LIN RI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, J8 SIM800L module: VCC GND TXD R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, J9 TP4056 module: B+ B- OUT+ OUT-, M1 coin vibration motor (seat), Q1 2N2222 (vibration driver), SW1 green button, SW2 red button, SW3 SOS button, SW4 power switch, SW5 tablet-drawer microswitch, U1 MCP6002, U2 INA126, U3 74HC4053 (body / R5 select), U4 74HC4052 (current pair), U5 74HC4052 (sense pair), U6 ESP32-WROOM-32 (DevKit), U7 3.3 V LDO (on DevKit)

Commit message: Add spectroscopy (C1), self-calibrating reference (C2), patient-safety analysis (C3)
- 5/20/50 kHz leg spectroscopy with closed-form Cole fit (EWI); engine v3 frozen at T=7.0
- Rcal 0.1% reference on the spare 74HC4053 switch, ratio check + service SMS
- IEC 60601-1 type-BF single-fault simulation: all pass, >=12.8x margin
- Firmware DMA ADC, SIL emulator 31/31, schematic, guides, docs regenerated
Parts:
- added R22: 100 0.1% (Rcal), symbol Device:R
- R5: value 220 1% -> 120
- U3: value 74HC4053 (body / R5 select) -> 74HC4053 (body / reference / self-cal)
Connections:
- net GND: no longer U3.9 (S3)
- net RET: now also U3.5 (C0); no longer U3.13 (A1)
- net VREF: now also R22.2; no longer R5.2
- net CAL_SEL: now reaches U6.14 (IO12)
- net CAL_SEL: now also U3.9 (S3)
- net NCAL: now reaches U3.3 (C1)
- net NCAL: now also R5.2, R22.1
- net RTAP: now reaches U3.4 (C)
- net RTAP: now also U3.13 (A1)
- no-connect marks 14 -> 10

Commit message: Add CHARGE / USE safety switch (charger isolation)
- SW6 DPDT cuts both USB charger wires in USE; GPIO39 senses CHARGE and the firmware refuses to measure
- charger_leakage.py: earthed patient leakage 339 uA (cheap charger) / 72 mA (failed) without it, 0.19 uA in USE
- Schematic with netlist checks (ERC 0), parts list +Rs 50 (Rs 4,820, Rs 180 under the limit), guides and PDFs
- Firmware emulator check: no excitation while on CHARGE (33/33); voice clip added
Parts:
- removed J9: TP4056 module: B+ B- OUT+ OUT-, symbol Connector_Generic:Conn_01x04
- added J12: USB-C charge socket (5V, GND); the TP4056 own USB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, symbol Connector_Generic:Conn_01x02
- added J9: TP4056 module: IN+ IN- B+ B- OUT+ OUT-, symbol Connector_Generic:Conn_01x06
- added R23, R24: 100k, symbol Device:R
- added SW6: CHARGE / USE slide switch: USE cuts BOTH charger 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, symbol Switch:SW_DPDT_x2
- J11: value AD8232 (optional; off for pacemaker/ICD; LO- unused) -> AD8232 (optional; off for pacemaker/ICD; LO+/LO- unused)
Connections:
- net BAT_P: now also J9.3 (Pin_3)
- net GND: now also J9.2 (Pin_2), J9.4 (Pin_4), J9.6 (Pin_6), R24.2, SW6.5 (B)
- net VBAT_RAW: now also J9.5 (Pin_5)
- net ECG_LOP: no longer names the net of J11.4 (Pin_4)
- net ECG_LOP: no longer U6.5 (SENSOR_VN)
- new net CHG_IN: J9.1 (Pin_1), R23.1, SW6.2 (B)
- new net CHG_SENSE: R23.2, R24.1, U6.5 (SENSOR_VN)
- new net USB_5V: J12.1 (Pin_1), SW6.1 (A)
- new net USB_GND: J12.2 (Pin_2), SW6.4 (A)
- no-connect marks 10 -> 13
